Commit message: feat: enhance xarm_lite robot model with kinematics and semantic description

File: ws/src/multi_arm_sim/urdf/xarm_lite.urdf (robot description, URDF)
Before this commit: robot xarm_lite, 2 links, 1 joints
Links:
- added link elbow; visual cylinder length=0.25 radius=0.03
- added link end_effector; visual box size=0.05 0.05 0.05
- added link extruder
- added link shoulder; visual cylinder length=0.3 radius=0.04
- added link wrist; visual cylinder length=0.2 radius=0.02
Joints:
- added joint ee_joint: type fixed, parent wrist, child end_effector, origin xyz=0 0 0.2 rpy=0 0 0
- added joint elbow_joint: type revolute, parent shoulder, child elbow, origin xyz=0 0 0.3 rpy=0 0 0, axis 0 1 0, limit lower=-1.57 upper=1.57 effort=10 velocity=1
- added joint extruder_joint: type fixed, parent end_effector, child extruder, origin xyz=0 0 0.05 rpy=0 0 0
- added joint shoulder_joint: type revolute, parent arm_base, child shoulder, origin xyz=0 0 0.1 rpy=0 0 0, axis 0 1 0, limit lower=-3.14 upper=3.14 effort=10 velocity=1
- added joint wrist_joint: type revolute, parent elbow, child wrist, origin xyz=0 0 0.25 rpy=0 0 0, axis 0 1 0, limit lower=-3.14 upper=3.14 effort=10 velocity=1
